Commit message: updated humanoid urdf

File: urdf/humanoid_walker.urdf (robot description, URDF)
Before this commit: robot KneedCompassGait, 23 links, 22 joints
Links:
- removed link head
- removed link head_mass
- link torso: geometry visual cylinder length=0.6 radius=0.005
Joints:
- removed joint head_mass_weld
- removed joint torso_head_weld
- joint left_shoulder_pin: origin xyz=0 0 0.8 rpy=3.14159 0 0 -> xyz=0 0 0.6 rpy=3.14159 0 0
- joint right_shoulder_pin: origin xyz=0 0 0.8 rpy=3.14159 0 0 -> xyz=0 0 0.6 rpy=3.14159 0 0
- joint torso_mass_weld: origin xyz=0 0 0.4 -> xyz=0 0 0.3
